Commit message: feat(nav): 重构仿真环境与机器人模型，导航栈首次 8/8 全绿
大改环境与小车模型，修复一系列导致导航失败的连锁问题。
核心结论：8 目标连续导航从 0/8 提升到 8/8，真值误差 0.08~0.37m。

环境（worlds/ + tools/gen_world.py）
- 门洞 1.10 -> 1.90m。膨胀半径 0.35 下可用宽度 = 1.90 - 2*0.35 = 1.20m，
  原 1.10m 门洞扣掉膨胀后实际不可通行
- room_c 货架后移到 y in [3.10,4.90]。原位置距 x=-2.8 门洞中心线仅 0.18m，
  膨胀后封死门洞上沿，可用通道只剩 0.5m，机器人卡在门口
- 统一墙体/底座的高度分层，供地图生成按激光高度过滤

机器人（urdf/advanced_robot.urdf）
- 底盘 0.52x0.32x0.16，轮子 0.20 半轮距，消除驱动轮与底盘的几何嵌入
  （原轮子嵌进底板，转向时持续刮擦，实测错误率 12%）
- 万向球摩擦 mu 0.001 -> 各向异性 (mu1=0.02, mu2=0.25)。
  原值近乎无摩擦，机器人靠两个无阻力球支点原地打转，
  转 180 度实际只转 172 度
- 驱动轮接触 kp 1e6 -> 8e4，kd 1 -> 20，消除接触高频弹跳
- 补 libgazebo_ros_laser.so 转换插件。/scan 此前完全没有数据
- publishWheelTF=false，轮子 TF 交给 robot_state_publisher，消除
  TF_REPEATED_DATA 刷屏
- wheelSeparation 标定为几何真值 0.42（非补偿值）：
  修好物理阻力后，0.42 使 odom/truth 达到 1.0003 / 0.9959 / 1.0006。
  教训写在文件注释里：车体转不够与里程计虚报同时出现时，
  不能用 wheelSeparation 做补偿，那只是把误差换个方向

代价地图（config/）
- obstacle_layer/track_unknown_space: false，局部地图顶层
  track_unknown_space: false。此前恢复行为报
  "potential collision, Cost: -1.00"（-1 是 NO_INFORMATION 而非障碍），
  导致所有恢复手段连锁失效
- transform_tolerance 1.0 -> 0.25，footprint 与 base_footprint 对齐

规划器（config/）
- 保持 base_local_planner/TrajectoryPlannerROS。曾评估
  dwa_local_planner/DWAPlannerROS 以解决「背对目标时输出零速」的死锁，
  但整场景实测更差（1/8 通过，起步慢约 5 倍，恢复行为触发 11 次，
  把 AMCL 带偏到 4.25m），故保留 TPR 并在其参数文件里记录对比数据
- 新增 config/dwa_local_planner_params.yaml 保留完整 DWA 配置作对照
- latch_xy_goal_tolerance=false 并注明不可开启。设为 true 时会形成
  静默永久死锁：cmd_vel 持续 15Hz 输出但速度恒为 0，日志无任何报错

语义地点（config/locations.yaml）
- 全部重新选取，净空从 0.71~1.92 提升到 1.14~2.25（理论下限 0.712，
  实践下限 0.95）
- 同时按「门洞通道带」优化：穿 x=+-2.8 墙时可用 y 仅 [1.25,2.35]，
  原 room_a 在 y=2.54 必须先南绕 0.7m 才能出门，是失败高发点
- home(0,-3.40) corridor(0,-1.20) room_a(-3.90,1.80) room_c(0,2.20)
  room_b(4.45,1.20) room_d(-3.65,-2.45) hall(3.35,-3.10)

launch/
- gazebo.launch 接收并透传 yaw 参数。原硬编码 -Y 0，导致机器人朝 +X
  生成而 AMCL 认为朝 +Y（差 90 度），出现「导航成功但真值差数米」

新增工具
- tools/check_locations.py：地点体检。校验净空、给出最近障碍物、
  并用膨胀栅格 + A* 检查全部地点两两双向可达。
  能在启动 Gazebo 之前发现绝大多数导航问题

文档
- docs/VERIFY.md：完整自验证手册。含五分钟快速验证、8 目标回归脚本、
  按症状分类的故障排查（A~G）、设计约束与一键自查清单

其他
- .gitattributes 固定 ROS 相关文件为 LF。core.autocrlf=true 会让
  检出时转成 CRLF，导致 .sh 在 bash 里报 \r: command not found
- scripts/ 改用 parse_known_args，避免 roslaunch 注入的额外参数报错

File: robot_ws/src/llm_robot_agent/urdf/advanced_robot.urdf (robot description, URDF)
Before this commit: robot advanced_robot, 8 links, 7 joints
Links:
- removed link left_front_wheel
- removed link left_rear_wheel
- removed link right_front_wheel
- removed link right_rear_wheel
- added link base_footprint
- added link caster_front, mass 0.08; collision sphere radius=0.035; visual sphere radius=0.035
- added link caster_rear, mass 0.08; collision sphere radius=0.035; visual sphere radius=0.035
- added link chassis_trim; visual box size=0.53 0.33 0.02
- added link left_wheel, mass 0.35; collision cylinder length=0.06 radius=0.08; visual cylinder length=0.06 radius=0.08
- added link right_wheel, mass 0.35; collision cylinder length=0.06 radius=0.08; visual cylinder length=0.06 radius=0.08
- link base_link: mass 3.0 -> 4.0; geometry collision box size=0.52 0.32 0.16; visual box size=0.52 0.32 0.16
- link camera_link: mass 0.15 -> 0.10; geometry collision box size=0.06 0.10 0.05; visual box size=0.06 0.10 0.05
- link laser_link: mass 0.2 -> 0.18; geometry collision cylinder length=0.05 radius=0.045; visual cylinder length=0.05 radius=0.045
- link sensor_platform: mass 0.5 -> 0.30; geometry collision cylinder length=0.05 radius=0.09; visual cylinder length=0.05 radius=0.09
Joints:
- removed joint left_front_joint
- removed joint left_rear_joint
- removed joint right_front_joint
- removed joint right_rear_joint
- added joint base_footprint_joint: type fixed, parent base_footprint, child base_link, origin xyz=0 0 0.10
- added joint caster_front_joint: type fixed, parent base_link, child caster_front, origin xyz=0.22 0 -0.065
- added joint caster_rear_joint: type fixed, parent base_link, child caster_rear, origin xyz=-0.22 0 -0.065
- added joint chassis_trim_joint: type fixed, parent base_link, child chassis_trim
- added joint left_wheel_joint: type continuous, parent base_link, child left_wheel, origin xyz=0 0.20 -0.02, axis 0 1 0
- added joint right_wheel_joint: type continuous, parent base_link, child right_wheel, origin xyz=0 -0.20 -0.02, axis 0 1 0
- joint camera_joint: origin xyz=0.1 0 0.03 -> xyz=0.09 0 0.025
- joint sensor_platform_joint: origin xyz=0 0 0.1 -> xyz=0 0 0.16
